File: hardware/Pasta-Pounder-I/Pasta-Pounder-I.kicad_sch (KiCad schematic)
At the start: 38 parts, among them CN1 XT30UPB-M, J1 USB_C_Receptacle, J2 Brushed_Motor_1, J3 Brushed_Motor_2, Q1 AO3401A, SW1 RESET-SW, SW2 BOOT-SW, SW3 5.8 ZSPT, U1 DRV8874PWPR, U2 DRV8874PWPR, U4 USBLC6-2P6, U5 ESP32S3W1

Commit message: Finished Power Management Schematic
Parts:
- added C20, C26: 10uF,25V, PCM_JLCPCB:C_0603, symbol Device:C
- added C21, C27: 100nF, PCM_JLCPCB:C_0402, symbol Device:C
- added C22, C28: 10pF, PCM_JLCPCB:C_0402, symbol Device:C
- added C23, C29: 10uF, PCM_JLCPCB:C_0603, symbol Device:C
- added L2, L3: 4.7uH, lcsc_footprints:C98354_IND-SMD_L2_5-W2_0_WPN252012H, symbol Device:L
- added R12: 68kΩ, PCM_JLCPCB:R_0402, symbol Device:R
- added R13: 15kΩ, PCM_JLCPCB:R_0402, symbol Device:R
- added R14: 36kΩ, PCM_JLCPCB:R_0402, symbol Device:R
- added R15: 4k7Ω, PCM_JLCPCB:R_0402, symbol Device:R
- added U6, U7: SY8113BADC, lcsc_footprints:C78989_TSOT-23-6_L2_9-W1_6-P0_95-LS2_8-BR, symbol lcsc_imported:SY8113BADC
Connections:
- net +3V3: now also C28.2, C29.2, L3.2, R12.1
- net DRV1-EN: now also U5.39 (IO1)
- net DRV1-IPROPI: now also U5.5 (IO5)
- net DRV1-PH: now also U5.38 (IO2)
- net DRV1-nFAULT: now also U5.4 (IO4)
- net DRV1-nSLEEP: now also U5.15 (IO3)
- net DRV2-EN: now also U5.6 (IO6)
- net DRV2-IPROPI: now also U5.18 (IO10)
- net DRV2-PH: now also U5.7 (IO7)
- net DRV2-nFAULT: now also U5.17 (IO9)
- net DRV2-nSLEEP: now also U5.12 (IO8)
- net GND: now also C20.1, C23.1, C26.1, C29.1, R13.2, R15.2, U6.2 (GND), U7.2 (GND)
- net VCC: now also C20.2, C26.2, U6.4 (EN), U6.5 (IN), U7.4 (EN), U7.5 (IN)
- new net: C22.1, R14.2, R15.1, U6.3 (FB)
- new net: C28.1, R12.2, R13.1, U7.3 (FB)
- new net: C27.1, U7.1 (BS)
- new net: C27.2, L3.1, U7.6 (LX)
- new net: C21.1, U6.1 (BS)
- new net: C21.2, L2.1, U6.6 (LX)
- new net +5V: C22.2, C23.2, L2.2, R14.1
- no-connect marks 47 -> 37
Other:
- note added: "3V3 Buck Converter"
- note added: "5V Buck Converter"
- note added: "Ref Pwr"
